File: pcb/v1.1/rv1106.kicad_pcb (KiCad board)
At the start: 4 copper layers, 86 x 56 mm, 217 parts, among them J1 GPIO, J201 Micro_SD_Card_Det1, J301 USB_C_Receptacle_USB2.0_14P, J302 HR913129AE, J303 USB_A_Stacked, J304 USB_A_Stacked, J501 AudioJack, J502 Camera, Q501 FDG1024NZ, SW1 Boot, SW2 Reset, SW301 USB_Select, U1 RV1106G3, U101 EA3036CQB, U102 PAM2306AYPAA, U202 Flash, U302 FSUSB42MUX, U303 CH334F, U402 ESP32-C6-MINI-1, U501 LSM6DSR, Y1 32.768kHz, Y2 24MHz 20ppm, Y301 12MHz

Commit message: Update docs
Parts:
- R3, R4, R5, R6: value 1k -> 10k
- R301, R302: value 22 -> 10
- R309: value 1k -> 10
- RN301, RN302, RN303: value 22 -> 0
